Commit message: Add 6 wheel robot urdf core

File: src/examplo_bot/description/core/robot_core.xacro (robot description, xacro)
@@ -18,108 +18,192 @@
     </link>
     <!-- CHASSIS LINK -->
+    <xacro:property name="chassis_length" value="0.7" />
+    <xacro:property name="chassis_width" value="0.65" />
+    <xacro:property name="chassis_height" value="0.1" />
     <joint name="chassis_joint" type="fixed">
         <parent link="base_link"/>
-        <child link="chassis"/>
-        <origin xyz="-0.1 0 0"/>
-    </joint>
-    <link name="chassis">
-        <visual>
-            <origin xyz="0.15 0 0.075"/>
-            <geometry>
-                <box size="0.3 0.3 0.15"/>
+        <child link="chassis_link"/>
+        <origin xyz="0 0 0"/>
+    </joint>
+    <link name="chassis_link">
+        <visual>
+            <origin xyz="0 0 0"/>
+            <geometry>
+                <box size="${chassis_length} ${chassis_width} ${chassis_height}"/>
             </geometry>
             <material name="white"/>
         </visual>
         <collision>
-            <origin xyz="0.15 0 0.075"/>
-            <geometry>
-                <box size="0.3 0.3 0.15"/>
-            </geometry>
-        </collision>
-        <xacro:inertial_box mass="0.5" x="0.3" y="0.3" z="0.15">
-            <origin xyz="0.15 0 0.075" rpy="0 0 0"/>
+            <origin xyz="0 0 0"/>
+            <geometry>
+                <box size="${chassis_length} ${chassis_width} ${chassis_height}"/>
+            </geometry>
+        </collision>
+        <xacro:inertial_box mass="1" x="${chassis_length}" y="${chassis_width}" z="${chassis_height}">
+            <origin xyz="0 0 0" rpy="0 0 0"/>
         </xacro:inertial_box>
     </link>
-    <gazebo reference="chassis">
+    <gazebo reference="chassis_link">
         <material>Gazebo/White</material>
     </gazebo>
-    <!-- LEFT WHEEL LINK -->
-    <joint name="left_wheel_joint" type="continuous">
-        <parent link="base_link"/>
-        <child link="left_wheel"/>
-        <origin xyz="0 0.175 0" rpy="-${pi/2} 0 0" />
+    <!-- WHEEL PROPERTIES -->
+    <xacro:property name="wheel_radius" value="0.09" />
+    <xacro:property name="wheel_thickness" value="0.04" />
+    <xacro:property name="wheel_seperation" value="0.21" />
+    <!-- WHEEL LINKS LEFT 1 -->
+    <joint name="left_wheel_1_joint" type="continuous">
+        <parent link="base_link"/>
+        <child link="left_wheel_1_link"/>
+        <origin xyz="${wheel_seperation} ${chassis_width/2 + wheel_thickness/2} 0" rpy="-${pi/2} 0 0" />
         <axis xyz="0 0 1"/>
     </joint>
-    <link name="left_wheel">
-        <visual>
-            <geometry>
-                <cylinder radius="0.05" length="0.04"/>
-            </geometry>
-            <material name="blue"/>
-        </visual>
-        <collision>
-            <geometry>
-                <cylinder radius="0.05" length="0.04"/>
-            </geometry>
-        </collision>
-        <xacro:inertial_cylinder mass="0.1" length="0.04" radius="0.05">
-            <origin xyz="0 0 0" rpy="0 0 0"/>
-        </xacro:inertial_cylinder>
-    </link>
-    <gazebo reference="left_wheel">
-        <material>Gazebo/Blue</material>
-    </gazebo>
-    <!-- RIGHT WHEEL LINK -->
-    <joint name="right_wheel_joint" type="continuous">
-        <parent link="base_link"/>
-        <child link="right_wheel"/>
-        <origin xyz="0 -0.175 0" rpy="${pi/2} 0 0" />
+    <link name="left_wheel_1_link">
+        <visual>
+            <geometry>
+                <cylinder radius="${wheel_radius}" length="${wheel_thickness}"/>
+            </geometry>
+            <material name="blue"/>
+        </visual>
+        <collision>
+            <geometry>
+                <cylinder radius="${wheel_radius}" length="${wheel_thickness}"/>
+            </geometry>
+        </collision>
+        <xacro:inertial_cylinder mass="0.2" length="${wheel_thickness}" radius="${wheel_thickness}">
+            <origin xyz="0 0 0" rpy="0 0 0"/>
+        </xacro:inertial_cylinder>
+    </link>
+    <gazebo reference="left_wheel_1_link">
+        <material>Gazebo/Blue</material>
+    </gazebo>
+    <!-- WHEEL LINKS LEFT 2 -->
+    <joint name="left_wheel_2_joint" type="continuous">
+        <parent link="base_link"/>
+        <child link="left_wheel_2_link"/>
+        <origin xyz="0 ${chassis_width/2 + wheel_thickness/2} 0" rpy="-${pi/2} 0 0" />
+        <axis xyz="0 0 1"/>
+    </joint>
+    <link name="left_wheel_2_link">
+        <visual>
+            <geometry>
+                <cylinder radius="${wheel_radius}" length="${wheel_thickness}"/>
+            </geometry>
+            <material name="blue"/>
+        </visual>
+        <collision>
+            <geometry>
+                <cylinder radius="${wheel_radius}" length="${wheel_thickness}"/>
+            </geometry>
+        </collision>
+        <xacro:inertial_cylinder mass="0.2" length="${wheel_thickness}" radius="${wheel_thickness}">
+            <origin xyz="0 0 0" rpy="0 0 0"/>
+        </xacro:inertial_cylinder>
+    </link>
+    <gazebo reference="left_wheel_2_link">
+        <material>Gazebo/Blue</material>
+    </gazebo>
+    <!-- WHEEL LINKS LEFT 3 -->
+    <joint name="left_wheel_3_joint" type="continuous">
+        <parent link="base_link"/>
+        <child link="left_wheel_3_link"/>
+        <origin xyz="-${wheel_seperation} ${chassis_width/2 + wheel_thickness/2} 0" rpy="-${pi/2} 0 0" />
+        <axis xyz="0 0 1"/>
+    </joint>
+    <link name="left_wheel_3_link">
+        <visual>
+            <geometry>
+                <cylinder radius="${wheel_radius}" length="${wheel_thickness}"/>
+            </geometry>
+            <material name="blue"/>
+        </visual>
+        <collision>
+            <geometry>
+                <cylinder radius="${wheel_radius}" length="${wheel_thickness}"/>
+            </geometry>
+        </collision>
+        <xacro:inertial_cylinder mass="0.2" length="${wheel_thickness}" radius="${wheel_thickness}">
+            <origin xyz="0 0 0" rpy="0 0 0"/>
+        </xacro:inertial_cylinder>
+    </link>
+    <gazebo reference="left_wheel_3_link">
+        <material>Gazebo/Blue</material>
+    </gazebo>
+    <!-- WHEEL LINKS RIGHT 1 -->
+    <joint name="right_wheel_1_joint" type="continuous">
+        <parent link="base_link"/>
+        <child link="right_wheel_1_link"/>
+        <origin xyz="${wheel_seperation} -${chassis_width/2 + wheel_thickness/2} 0" rpy="${pi/2} 0 0" />
         <axis xyz="0 0 -1"/>
     </joint>
-    <link name="right_wheel">
-        <visual>
-            <geometry>
-                <cylinder radius="0.05" length="0.04"/>
-            </geometry>
-            <material name="blue"/>
-        </visual>
-        <collision>
-            <geometry>
-                <cylinder radius="0.05" length="0.04"/>
-            </geometry>
-        </collision>
-        <xacro:inertial_cylinder mass="0.1" length="0.04" radius="0.05">
-            <origin xyz="0 0 0" rpy="0 0 0"/>
-        </xacro:inertial_cylinder>
-    </link>
-    <gazebo reference="right_wheel">
-        <material>Gazebo/Blue</material>
-    </gazebo>
-    <!-- CASTER WHEEL LINK -->
-    <joint name="caster_wheel_joint" type="fixed">
-        <parent link="chassis"/>
-        <child link="caster_wheel"/>
-        <origin xyz="0.24 0 0"/>
-    </joint>
-    <link name="caster_wheel">
-        <visual>
-            <geometry>
-                <sphere radius="0.05"/>
-            </geometry>
-            <material name="black"/>
-        </visual>
-        <collision>
-            <geometry>
-                <sphere radius="0.05"/>
-            </geometry>
-        </collision>
-        <xacro:inertial_sphere mass="0.1" radius="0.05">
-            <origin xyz="0 0 0" rpy="0 0 0"/>
-        </xacro:inertial_sphere>
-    </link>
-    <gazebo reference="caster_wheel">
-        <material>Gazebo/Black</material>
-        <mu1 value="0.001"/>
-        <mu2 value="0.001"/>
+    <link name="right_wheel_1_link">
+        <visual>
+            <geometry>
+                <cylinder radius="${wheel_radius}" length="${wheel_thickness}"/>
+            </geometry>
+            <material name="blue"/>
+        </visual>
+        <collision>
+            <geometry>
+                <cylinder radius="${wheel_radius}" length="${wheel_thickness}"/>
+            </geometry>
+        </collision>
+        <xacro:inertial_cylinder mass="0.2" length="${wheel_thickness}" radius="${wheel_radius}">
+            <origin xyz="0 0 0" rpy="0 0 0"/>
+        </xacro:inertial_cylinder>
+    </link>
+    <gazebo reference="right_wheel_1_link">
+        <material>Gazebo/Blue</material>
+    </gazebo>
+    <!-- WHEEL LINKS RIGHT 2 -->
+    <joint name="right_wheel_2_joint" type="continuous">
+        <parent link="base_link"/>
+        <child link="right_wheel_2_link"/>
+        <origin xyz="0 -${chassis_width/2 + wheel_thickness/2} 0" rpy="${pi/2} 0 0" />
+        <axis xyz="0 0 -1"/>
+    </joint>
+    <link name="right_wheel_2_link">
+        <visual>
+            <geometry>
+                <cylinder radius="${wheel_radius}" length="${wheel_thickness}"/>
+            </geometry>
+            <material name="blue"/>
+        </visual>
+        <collision>
+            <geometry>
+                <cylinder radius="${wheel_radius}" length="${wheel_thickness}"/>
+            </geometry>
+        </collision>
+        <xacro:inertial_cylinder mass="0.2" length="${wheel_thickness}" radius="${wheel_radius}">
+            <origin xyz="0 0 0" rpy="0 0 0"/>
+        </xacro:inertial_cylinder>
+    </link>
+    <gazebo reference="right_wheel_2_link">
+        <material>Gazebo/Blue</material>
+    </gazebo>
+    <!-- WHEEL LINKS RIGHT 3 -->
+    <joint name="right_wheel_3_joint" type="continuous">
+        <parent link="base_link"/>
+        <child link="right_wheel_3_link"/>
+        <origin xyz="-${wheel_seperation} -${chassis_width/2 + wheel_thickness/2} 0" rpy="${pi/2} 0 0" />
+        <axis xyz="0 0 -1"/>
+    </joint>
+    <link name="right_wheel_3_link">
+        <visual>
+            <geometry>
+                <cylinder radius="${wheel_radius}" length="${wheel_thickness}"/>
+            </geometry>
+            <material name="blue"/>
+        </visual>
+        <collision>
+            <geometry>
+                <cylinder radius="${wheel_radius}" length="${wheel_thickness}"/>
+            </geometry>
+        </collision>
+        <xacro:inertial_cylinder mass="0.2" length="${wheel_thickness}" radius="${wheel_radius}">
+            <origin xyz="0 0 0" rpy="0 0 0"/>
+        </xacro:inertial_cylinder>
+    </link>
+    <gazebo reference="right_wheel_3_link">
+        <material>Gazebo/Blue</material>
     </gazebo>
 </robot>

Commit message: Setup diffdrive controller

File: src/examplo_bot/description/core/robot_core.xacro (robot description, xacro)
@@ -2,59 +2,58 @@
 <robot xmlns:xacro="http://www.ros.org/wiki/xacro" >
     <xacro:include filename="macros.xacro"/>
-    <material name="white">
-        <color rgba="1 1 1 1" />
-    </material>
-    <material name="orange">
-        <color rgba="1 0.3 0.1 1"/>
-    </material>
-    <material name="blue">
-        <color rgba="0.2 0.2 1 1"/>
-    </material>
-    <material name="black">
-        <color rgba="0 0 0 1"/>
-    </material>
-    <!-- BASE LINK -->
-    <link name="base_link">
-    </link>
-    <!-- CHASSIS LINK -->
+    <!-- PROPERTIES -->
     <xacro:property name="chassis_length" value="0.7" />
     <xacro:property name="chassis_width" value="0.65" />
     <xacro:property name="chassis_height" value="0.1" />
-    <joint name="chassis_joint" type="fixed">
-        <parent link="base_link"/>
-        <child link="chassis_link"/>
-        <origin xyz="0 0 0"/>
-    </joint>
-    <link name="chassis_link">
-        <visual>
-            <origin xyz="0 0 0"/>
-            <geometry>
-                <box size="${chassis_length} ${chassis_width} ${chassis_height}"/>
-            </geometry>
-            <material name="white"/>
-        </visual>
-        <collision>
-            <origin xyz="0 0 0"/>
-            <geometry>
-                <box size="${chassis_length} ${chassis_width} ${chassis_height}"/>
-            </geometry>
-        </collision>
-        <xacro:inertial_box mass="1" x="${chassis_length}" y="${chassis_width}" z="${chassis_height}">
-            <origin xyz="0 0 0" rpy="0 0 0"/>
-        </xacro:inertial_box>
-    </link>
-    <gazebo reference="chassis_link">
-        <material>Gazebo/White</material>
-    </gazebo>
-    <!-- WHEEL PROPERTIES -->
     <xacro:property name="wheel_radius" value="0.09" />
     <xacro:property name="wheel_thickness" value="0.04" />
     <xacro:property name="wheel_seperation" value="0.21" />
-    <!-- WHEEL LINKS LEFT 1 -->
-    <joint name="left_wheel_1_joint" type="continuous">
+    <material name="white">
+        <color rgba="1 1 1 1" />
+    </material>
+    <material name="orange">
+        <color rgba="1 0.3 0.1 1"/>
+    </material>
+    <material name="blue">
+        <color rgba="0.2 0.2 1 1"/>
+    </material>
+    <material name="black">
+        <color rgba="0 0 0 1"/>
+    </material>
+    <!-- BASE LINK -->
+    <link name="base_link">
+    </link>
+    <!-- CHASSIS LINK -->
+    <joint name="chassis_joint" type="fixed">
+        <parent link="base_link"/>
+        <child link="chassis_link"/>
+        <origin xyz="0 0 0"/>
+    </joint>
+    <link name="chassis_link">
+        <visual>
+            <origin xyz="0 0 0"/>
+            <geometry>
+                <box size="${chassis_length} ${chassis_width} ${chassis_height}"/>
+            </geometry>
+            <material name="white"/>
+        </visual>
+        <collision>
+            <origin xyz="0 0 0"/>
+            <geometry>
+                <box size="${chassis_length} ${chassis_width} ${chassis_height}"/>
+            </geometry>
+        </collision>
+        <xacro:inertial_box mass="1" x="${chassis_length}" y="${chassis_width}" z="${chassis_height}">
+            <origin xyz="0 0 0" rpy="0 0 0"/>
+        </xacro:inertial_box>
+    </link>
+    <gazebo reference="chassis_link">
+        <material>Gazebo/White</material>
+    </gazebo>
+    <!-- WHEEL LINKS LEFT 1 (CASTER) -->
+    <joint name="left_wheel_1_joint" type="fixed">
         <parent link="base_link"/>
         <child link="left_wheel_1_link"/>
         <origin xyz="${wheel_seperation} ${chassis_width/2 + wheel_thickness/2} 0" rpy="-${pi/2} 0 0" />
-        <axis xyz="0 0 1"/>
     </joint>
     <link name="left_wheel_1_link">
@@ -76,4 +75,6 @@
     <gazebo reference="left_wheel_1_link">
         <material>Gazebo/Blue</material>
+        <mu1 value="0.001"/>
+        <mu2 value="0.001"/>
     </gazebo>
     <!-- WHEEL LINKS LEFT 2 -->
@@ -103,10 +104,9 @@
         <material>Gazebo/Blue</material>
     </gazebo>
-    <!-- WHEEL LINKS LEFT 3 -->
-    <joint name="left_wheel_3_joint" type="continuous">
+    <!-- WHEEL LINKS LEFT 3 (CASTER) -->
+    <joint name="left_wheel_3_joint" type="fixed">
         <parent link="base_link"/>
         <child link="left_wheel_3_link"/>
         <origin xyz="-${wheel_seperation} ${chassis_width/2 + wheel_thickness/2} 0" rpy="-${pi/2} 0 0" />
-        <axis xyz="0 0 1"/>
     </joint>
     <link name="left_wheel_3_link">
@@ -128,11 +128,12 @@
     <gazebo reference="left_wheel_3_link">
         <material>Gazebo/Blue</material>
-    </gazebo>
-    <!-- WHEEL LINKS RIGHT 1 -->
-    <joint name="right_wheel_1_joint" type="continuous">
+        <mu1 value="0.001"/>
+        <mu2 value="0.001"/>
+    </gazebo>
+    <!-- WHEEL LINKS RIGHT 1 (CASTER) -->
+    <joint name="right_wheel_1_joint" type="fixed">
         <parent link="base_link"/>
         <child link="right_wheel_1_link"/>
         <origin xyz="${wheel_seperation} -${chassis_width/2 + wheel_thickness/2} 0" rpy="${pi/2} 0 0" />
-        <axis xyz="0 0 -1"/>
     </joint>
     <link name="right_wheel_1_link">
@@ -154,4 +155,6 @@
     <gazebo reference="right_wheel_1_link">
         <material>Gazebo/Blue</material>
+        <mu1 value="0.001"/>
+        <mu2 value="0.001"/>
     </gazebo>
     <!-- WHEEL LINKS RIGHT 2 -->
@@ -181,10 +184,9 @@
         <material>Gazebo/Blue</material>
     </gazebo>
-    <!-- WHEEL LINKS RIGHT 3 -->
-    <joint name="right_wheel_3_joint" type="continuous">
+    <!-- WHEEL LINKS RIGHT 3 (CASTER) -->
+    <joint name="right_wheel_3_joint" type="fixed">
         <parent link="base_link"/>
         <child link="right_wheel_3_link"/>
         <origin xyz="-${wheel_seperation} -${chassis_width/2 + wheel_thickness/2} 0" rpy="${pi/2} 0 0" />
-        <axis xyz="0 0 -1"/>
     </joint>
     <link name="right_wheel_3_link">
@@ -206,4 +208,6 @@
     <gazebo reference="right_wheel_3_link">
         <material>Gazebo/Blue</material>
+        <mu1 value="0.001"/>
+        <mu2 value="0.001"/>
     </gazebo>
 </robot>

File: src/examplo_bot/description/sim.urdf.xacro (robot description, xacro)
@@ -2,3 +2,4 @@
 <robot xmlns:xacro="http://www.ros.org/wiki/xacro"  name="examplo_bot_sim">
     <xacro:include filename="core/robot_core.xacro" />
+    <xacro:include filename="controlsim.xacro" />
 </robot>
